Commit message: moveit config

File: kuka_kr6_description/urdf/kuka_kr6.xacro (robot description, xacro)
@@ -40,5 +40,5 @@
         <geometry>
           <mesh
-            filename="package://kuka_description/meshes/visual/base_link.stl" />
+            filename="package://kuka_kr6_description/meshes/visual/base_link.stl" />
         </geometry>
         <material name="Grey1" />
@@ -50,5 +50,5 @@
         <geometry>
           <mesh
-            filename="package://kuka_description/meshes/collision/base_link.stl" />
+            filename="package://kuka_kr6_description/meshes/collision/base_link.stl" />
         </geometry>
       </collision>
@@ -91,15 +91,15 @@
         <geometry>
           <mesh
-            filename="package://kuka_description/meshes/visual/link_1.stl" />
-        </geometry>
-        <material name="KUKA_Orange" />
-      </visual>
-      <collision>
-        <origin
-          xyz="0 0 0"
-          rpy="0 0 0" />
-        <geometry>
-          <mesh
-            filename="package://kuka_description/meshes/collision/link_1.stl" />
+            filename="package://kuka_kr6_description/meshes/visual/link_1.stl" />
+        </geometry>
+        <material name="KUKA_Orange" />
+      </visual>
+      <collision>
+        <origin
+          xyz="0 0 0"
+          rpy="0 0 0" />
+        <geometry>
+          <mesh
+            filename="package://kuka_kr6_description/meshes/collision/link_1.stl" />
         </geometry>
       </collision>
@@ -143,15 +143,15 @@
         <geometry>
           <mesh
-            filename="package://kuka_description/meshes/visual/link_2.stl" />
-        </geometry>
-        <material name="KUKA_Orange" />
-      </visual>
-      <collision>
-        <origin
-          xyz="0 0 0"
-          rpy="0 0 0" />
-        <geometry>
-          <mesh
-            filename="package://kuka_description/meshes/collision/link_2.stl" />
+            filename="package://kuka_kr6_description/meshes/visual/link_2.stl" />
+        </geometry>
+        <material name="KUKA_Orange" />
+      </visual>
+      <collision>
+        <origin
+          xyz="0 0 0"
+          rpy="0 0 0" />
+        <geometry>
+          <mesh
+            filename="package://kuka_kr6_description/meshes/collision/link_2.stl" />
         </geometry>
       </collision>
@@ -161,5 +161,5 @@
     <!-- Joint A3 -->
     <joint
-      name="${prefix}joint a3"
+      name="${prefix}joint_a3"
       type="revolute">
       <origin
@@ -195,15 +195,15 @@
         <geometry>
           <mesh
-            filename="package://kuka_description/meshes/visual/link_3.stl" />
-        </geometry>
-        <material name="KUKA_Orange" />
-      </visual>
-      <collision>
-        <origin
-          xyz="0 0 0"
-          rpy="0 0 0" />
-        <geometry>
-          <mesh
-            filename="package://kuka_description/meshes/collision/link_3.stl" />
+            filename="package://kuka_kr6_description/meshes/visual/link_3.stl" />
+        </geometry>
+        <material name="KUKA_Orange" />
+      </visual>
+      <collision>
+        <origin
+          xyz="0 0 0"
+          rpy="0 0 0" />
+        <geometry>
+          <mesh
+            filename="package://kuka_kr6_description/meshes/collision/link_3.stl" />
         </geometry>
       </collision>
@@ -246,15 +246,15 @@
         <geometry>
           <mesh
-            filename="package://kuka_description/meshes/visual/link_4.stl" />
-        </geometry>
-        <material name="KUKA_Orange" />
-      </visual>
-      <collision>
-        <origin
-          xyz="0 0 0"
-          rpy="0 0 0" />
-        <geometry>
-          <mesh
-            filename="package://kuka_description/meshes/collision/link_4.stl" />
+            filename="package://kuka_kr6_description/meshes/visual/link_4.stl" />
+        </geometry>
+        <material name="KUKA_Orange" />
+      </visual>
+      <collision>
+        <origin
+          xyz="0 0 0"
+          rpy="0 0 0" />
+        <geometry>
+          <mesh
+            filename="package://kuka_kr6_description/meshes/collision/link_4.stl" />
         </geometry>
       </collision>
@@ -297,15 +297,15 @@
         <geometry>
           <mesh
-            filename="package://kuka_description/meshes/visual/link_5.stl" />
-        </geometry>
-        <material name="KUKA_Orange" />
-      </visual>
-      <collision>
-        <origin
-          xyz="0 0 0"
-          rpy="0 0 0" />
-        <geometry>
-          <mesh
-            filename="package://kuka_description/meshes/collision/link_5.stl" />
+            filename="package://kuka_kr6_description/meshes/visual/link_5.stl" />
+        </geometry>
+        <material name="KUKA_Orange" />
+      </visual>
+      <collision>
+        <origin
+          xyz="0 0 0"
+          rpy="0 0 0" />
+        <geometry>
+          <mesh
+            filename="package://kuka_kr6_description/meshes/collision/link_5.stl" />
         </geometry>
       </collision>
@@ -348,5 +348,5 @@
         <geometry>
           <mesh
-            filename="package://kuka_description/meshes/visual/link_6.stl" />
+            filename="package://kuka_kr6_description/meshes/visual/link_6.stl" />
         </geometry>
         <material name="Grey3" />
@@ -358,7 +358,33 @@
         <geometry>
           <mesh
-            filename="package://kuka_description/meshes/collision/link_6.stl" />
-        </geometry>
-      </collision>
+            filename="package://kuka_kr6_description/meshes/collision/link_6.stl" />
+        </geometry>
+      </collision>
+    </link>
+    <!-- **************************************** -->
+    <!-- A6 -->
+    <!-- Tool joint -->
+    <joint
+      name="${prefix}joint_tool"
+      type="fixed">
+      <origin
+        xyz="0.1125 -0.02025 0"
+        rpy="0 0 0" />
+      <parent
+        link="${prefix}link_6" />
+      <child
+        link="${prefix}link_tool" />
+      <axis
+        xyz="1 0 0" />
+    </joint>
+    <!-- Tool link -->
+    <link name="${prefix}link_tool">
+      <inertial>
+        <origin
+          xyz="0 0 0"
+          rpy="0 0 0" />
+        <mass value="0.01" />
+        <simple_inertia_def diag="0.01"/>
+      </inertial>
     </link>
   </xacro:macro>
